File: Schematic/GBxCart_RW_v1.1_Schematic.sch (EAGLE design)
At the start: 31 parts, among them J1 AVR_SPI_6, J2 GB_CART1, J3 Mini USB, Q1 2N7002K (N), U1 MEGA32-A, U2 CH340G, U3 RT9013, U4 INVERTER, X1 8MHz, X2 12MHz

Commit message: Added GB Camera Saver program
GB Camera Saver
v1.0 – 12 July 2017
• Initial Release
Parts:
- removed Q1: 2N7002K (N), alex:2N7002K_(N)SOT-23
- removed U1: MEGA32-A, avr-5:MEGA32-A
- removed U4: INVERTER, SparkFun:INVERTER
- added IC1: ATMEGA8515L-8AU, avr-5:MEGA8515-A
- LED1: device adafruit:LEDCHIP-LED0805 -> adafruit:LEDCHIP-LED0805-NS
- LED2: value LED -> 3.3V LED; device adafruit:LEDCHIP-LED0805 -> adafruit:LEDCHIP-LED0805-NS
- LED3: value LED -> 5V LED; device adafruit:LEDCHIP-LED0805 -> adafruit:LEDCHIP-LED0805-NS
- R5: device adafruit:R-US_R0805_2 -> adafruit:R-US_R0603
Connections:
- removed net N$4: R4.1, U4.Y
- removed net N$6: LED3.C, Q1.D
- new net N$8: IC1.(RD)PD7, R2.1
- new net N$9: IC1.PE0(ICP/INT2), R4.1
- net *MREQ/CS: now also IC1.(XCK)PD4; no longer U1.(ICP)PD6
- net *RD: now also IC1.(OC1A)PD5; no longer U1.(OC1A)PD5
- net *RESET/CS2: now also IC1.PE2(OC1B); no longer U1.(OC2)PD7
- net *WR: now also IC1.(WR)PD6; no longer U1.(OC1B)PD4
- net 3.3V: no longer R2.1, U4.VCC
- net A0: now also IC1.(T0/OC0)PB0; no longer U1.(T0/XCK)PB0
- net A1: now also IC1.(T1)PB1; no longer U1.(T1)PB1
- net A10: now also IC1.(AD2)PA2; no longer U1.(ADC2)PA2
- net A11: now also IC1.(AD3)PA3; no longer U1.(ADC3)PA3
- net A12: now also IC1.(AD4)PA4; no longer U1.(ADC4)PA4
- net A13: now also IC1.(AD5)PA5; no longer U1.(ADC5)PA5
- net A14: now also IC1.(AD6)PA6; no longer U1.(ADC6)PA6
- net A15: now also IC1.(AD7)PA7; no longer U1.(ADC7)PA7
- net A2: now also IC1.(AIN0)PB2; no longer U1.(AIN0/INT2)PB2
- net A3: now also IC1.(AIN1)PB3; no longer U1.(AIN1/OC0)PB3
- net A4: now also IC1.(SS)PB4; no longer U1.(SS)PB4
- net A5/MOSI: now also IC1.(MOSI)PB5; no longer U1.(MOSI)PB5
- net A6/MISO: now also IC1.(MISO)PB6; no longer U1.(MISO)PB6
- net A7/SCK: now also IC1.(SCK)PB7; no longer U1.(SCK)PB7
- net A8: now also IC1.(AD0)PA0; no longer U1.(ADC0)PA0
- net A9: now also IC1.(AD1)PA1; no longer U1.(ADC1)PA1
- net ATMEGA_RXD: now also IC1.(RXD)PD0; no longer U1.(RXD)PD0
- net ATMEGA_TXD: now also IC1.(TXD)PD1; no longer U1.(TXD)PD1
- net AUDIO_IN: now also IC1.PE1(ALE)
- net D0: now also IC1.(A8)PC0; no longer U1.PC0(SCL)
- net D1: now also IC1.(A9)PC1; no longer U1.PC1(SDA)
- net D2: now also IC1.(A10)PC2; no longer U1.(TCK)PC2
- net D3: now also IC1.(A11)PC3; no longer U1.(TMS)PC3
- net D4: now also IC1.(A12)PC4; no longer U1.(TDO)PC4
- net D5: now also IC1.(A13)PC5; no longer U1.(TDI)PC5
- net D6: now also IC1.(A14)PC6; no longer U1.(TOSC1)PC6
- net D7: now also IC1.(A15)PC7; no longer U1.(TOSC2)PC7
- net GND: now also IC1.GND, LED3.C; no longer Q1.S, U1.AGND, U1.GND, U1.GND1, U1.GND2, U4.GND
- net N$1: now also IC1.(INT1)PD3; no longer U1.(INT1)PD3
- net RESET: now also IC1.RESET; no longer U1.RESET
- net SW_DT: now also IC1.(INT0)PD2; no longer Q1.G, U1.(INT0)PD2, U4.A
- net VCC: now also IC1.VCC; no longer U1.AVCC, U1.VCC, U1.VCC1, U1.VCC2
- net XTAL5: now also IC1.XTAL2; no longer U1.XTAL2
- net XTAL6: now also IC1.XTAL1; no longer U1.XTAL1
Other:
- note added: "GBxCart RW PCB v1.1 By insideGadgets"
- note added: "Voltage Reg and DPDT Switch"
- note removed: "Inverter for lighting 3.3V/5V LEDs"
- note removed: "Voltage Reg and 5V/3.3V Switch"
- moved on the sheet: C1, C11, C2, J2, LED2, LED3, R2, R3, R4, X1
